File: AREG.kicad_sch (KiCad schematic)
At the start: 9 parts, among them U1 AP63200WU-7

Commit message: Began board layout
Parts:
- added TP31, TP32, TP33, TP34: Test Point, TestPoint:TestPoint_THTPad_D1.0mm_Drill0.5mm, symbol Project_Components:Inline Test Point
- C14: renamed from C13; footprint (none) -> Capacitor_SMD:C_0603_1608Metric_Pad1.08x0.95mm_HandSolder
- C16: renamed from C14; footprint (none) -> Capacitor_SMD:C_0603_1608Metric_Pad1.08x0.95mm_HandSolder
- C18: renamed from C15; footprint (none) -> Capacitor_SMD:C_0603_1608Metric_Pad1.08x0.95mm_HandSolder
- C20: renamed from C16; footprint (none) -> Capacitor_SMD:C_0603_1608Metric_Pad1.08x0.95mm_HandSolder
- C22: renamed from C17; footprint (none) -> Capacitor_SMD:C_0603_1608Metric_Pad1.08x0.95mm_HandSolder
- L1: footprint (none) -> Inductor_SMD:L_0603_1608Metric_Pad1.05x0.95mm_HandSolder
- R15: renamed from R11; footprint (none) -> Resistor_SMD:R_0603_1608Metric_Pad0.98x0.95mm_HandSolder
- R16: renamed from R12; footprint (none) -> Resistor_SMD:R_0603_1608Metric_Pad0.98x0.95mm_HandSolder
- renumbered U1 to U4
Connections:
- net FB: now also TP31.1
- net VOUT: now also TP34.1
- net at C16.2, L1.1, U4.5 (SW): now also TP32.1
- net at C16.1, U4.6 (BST): now also TP33.1
